File: KiCAD/Blinker Fluid.kicad_sch (KiCad schematic)
At the start: 147 parts, among them J1 Conn_02x32_Counter_Clockwise, U1 74HCT574, U2 74HCT574, U3 74HCT574, U4 74HCT574, U5 74HCT574, U6 74HCT574, U7 74HCT574, U8 74HCT574, U9 NE555

Commit message: revised
Parts:
- C71: value 10uf -> 1uf; LCSC C7171 -> C1953183
- R72: value 10k -> 47k; LCSC C25744 -> C25762
Changed lines of the file:
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@@
 			)
 		)
-		(property "Value" "10k"
+		(property "Value" "47k"
 			(at 681.99 243.84 90)
 			(effects
@@
 			)
 		)
-		(property "LCSC" "C25744"
+		(property "LCSC" "C25762"
 			(at 680.466 243.84 0)
 			(effects
@@
 			)
 		)
-		(property "Value" "10uf"
+		(property "Value" "1uf"
 			(at 669.29 254.546 0)
 			(effects
@@
 			)
 		)
-		(property "LCSC" "C7171"
+		(property "LCSC" "C1953183"
 			(at 669.29 252.006 0)
 			(effects

Commit message: Updated 17-02-26
Parts:
- C72: footprint Capacitor_SMD:C_0402_1005Metric_Pad0.74x0.62mm_HandSolder -> Capacitor_SMD:C_0805_2012Metric_Pad1.18x1.45mm_HandSolder
- R1, R2, R3, R4, R5, R53, R54, R55, R56, R57, R58, R59, R60, R61, R62, R63: value 330 -> 620
- R10, R11, R12, R13, R14, R15, R17, R18, R19, R20, R21, R22, R23, R24, R25, R26, R27, R49, R6, R7, R8, R9: value 680 -> 470
- R29, R30, R31, R32, R33, R34, R35, R36, R37, R38, R39, R40, R41, R42, R43, R44, R45, R46, R47, R48, R50, R51, R52: value 470 -> 820
- R71: value 1k -> 10k; footprint Resistor_SMD:R_0402_1005Metric_Pad0.72x0.64mm_HandSolder -> Resistor_SMD:R_0805_2012Metric_Pad1.20x1.40mm_HandSolder
- R72: footprint Resistor_SMD:R_0402_1005Metric_Pad0.72x0.64mm_HandSolder -> Resistor_SMD:R_0805_2012Metric_Pad1.20x1.40mm_HandSolder
Changed lines of the file:
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@@
 			)
 		)
-		(property "Value" "680"
+		(property "Value" "470"
 			(at 509.27 382.27 90)
 			(effects
@@
 			)
 		)
-		(property "Value" "680"
+		(property "Value" "470"
 			(at 509.27 335.28 90)
 			(effects
@@
 			)
 		)
-		(property "Value" "330"
+		(property "Value" "620"
 			(at 716.28 337.82 90)
 			(effects
@@
 			)
 		)
-		(property "Value" "330"
+		(property "Value" "620"
 			(at 505.46 337.82 90)
 			(effects
@@
 			)
 		)
-		(property "Value" "680"
+		(property "Value" "470"
 			(at 505.46 332.74 90)
 			(effects
@@
 			)
 		)
-		(property "Value" "330"
+		(property "Value" "620"
 			(at 505.46 347.98 90)
 			(effects
@@
 			)
 		)
-		(property "Value" "470"
+		(property "Value" "820"
 			(at 709.93 391.16 90)
 			(effects
@@
 			)
 		)
-		(property "Value" "470"
+		(property "Value" "820"
 			(at 715.01 429.26 90)
 			(effects
@@
 			)
 		)
-		(property "Value" "680"
+		(property "Value" "470"
 			(at 505.46 389.89 90)
 			(effects
@@
 			)
 		)
-		(property "Value" "680"
+		(property "Value" "470"
 			(at 505.46 481.33 90)
 			(effects
@@
 			)
 		)
-		(property "Value" "330"
+		(property "Value" "620"
 			(at 711.2 335.28 90)
 			(effects
@@
 			)
 		)
-		(property "Value" "470"
+		(property "Value" "820"
 			(at 715.01 424.18 90)
 			(effects
@@
 			)
 		)
-		(property "Value" "470"
+		(property "Value" "820"
 			(at 715.01 434.34 90)
 			(effects
@@
 			)
 		)
-		(property "Value" "470"
+		(property "Value" "820"
 			(at 505.46 471.17 90)
 			(effects
@@
 			)
 		)
-		(property "Value" "680"
+		(property "Value" "470"
 			(at 737.87 386.08 90)
 			(effects
@@
 			)
 		)
-		(property "Value" "470"
+		(property "Value" "820"
 			(at 509.27 473.71 90)
 			(effects
@@
 			)
 		)
-		(property "Value" "330"
+		(property "Value" "620"
 			(at 715.01 381 90)
 			(effects
@@
 			)
 		)
-		(property "Value" "470"
+		(property "Value" "820"
 			(at 709.93 421.64 90)
 			(effects
@@
 			)
 		)
-		(property "Value" "330"
+		(property "Value" "620"
 			(at 711.2 330.2 90)
 			(effects
@@
 			)
 		)
-		(property "Value" "680"
+		(property "Value" "470"
 			(at 509.27 425.45 90)
 			(effects
@@
 			)
 		)
-		(property "Value" "330"
+		(property "Value" "620"
 			(at 716.28 342.9 90)
 			(effects
@@
 			)
 		)
-		(property "Value" "470"
+		(property "Value" "820"
 			(at 715.01 474.98 90)
 			(effects
@@
 			)
 		)
-		(property "Value" "330"
+		(property "Value" "620"
 			(at 711.2 378.46 90)
 			(effects
@@
 			)
 		)
-		(property "Value" "330"
+		(property "Value" "620"
 			(at 509.27 345.44 90)
 			(effects
@@
 			)
 		)
-		(property "Value" "680"
+		(property "Value" "470"
 			(at 509.27 483.87 90)
 			(effects
@@
 			)
 		)
-		(property "Value" "680"
+		(property "Value" "470"
 			(at 509.27 392.43 90)
 			(effects
@@
 			)
 		)
-		(property "Value" "470"
+		(property "Value" "820"
 			(at 715.01 388.62 90)
 			(effects
@@
 			)
 		)
-		(property "Value" "680"
+		(property "Value" "470"
 			(at 509.27 330.2 90)
 			(effects
@@
 			)
 		)
-		(property "Value" "680"
+		(property "Value" "470"
 			(at 509.27 435.61 90)
 			(effects
@@
 			)
 		)
-		(property "Value" "330"
+		(property "Value" "620"
 			(at 509.27 340.36 90)
 			(effects
@@
 			)
 		)
-		(property "Value" "330"
+		(property "Value" "620"
 			(at 711.2 345.44 90)
 			(effects
@@
 			)
 		)
-		(property "Value" "680"
+		(property "Value" "470"
 			(at 509.27 377.19 90)
 			(effects
@@
 			)
 		)
-		(property "Value" "470"
+		(property "Value" "820"
 			(at 709.93 472.44 90)
 			(effects
@@
 			)
 		)
-		(property "Value" "470"
+		(property "Value" "820"
 			(at 709.93 477.52 90)
 			(effects
@@
 			)
 		)
-		(property "Value" "470"
+		(property "Value" "820"
 			(at 715.01 469.9 90)
 			(effects
@@
 			)
 		)
-		(property "Value" "470"
+		(property "Value" "820"
 			(at 709.93 482.6 90)
 			(effects
@@
 			)
 		)
-		(property "Value" "680"
+		(property "Value" "470"
 			(at 505.46 433.07 90)
 			(effects
@@
 			)
 		)
-		(property "Value" "470"
+		(property "Value" "820"
 			(at 509.27 468.63 90)
 			(effects
@@
 			)
 		)
-		(property "Value" "680"
+		(property "Value" "470"
 			(at 505.46 438.15 90)
 			(effects
@@
 			)
 		)
-		(property "Value" "680"
+		(property "Value" "470"
 			(at 509.27 478.79 90)
 			(effects
@@
 			)
 		)
-		(property "Value" "470"
+		(property "Value" "820"
 			(at 715.01 485.14 90)
 			(effects
@@
 			)
 		)
-		(property "Value" "680"
+		(property "Value" "470"
 			(at 509.27 420.37 90)
 			(effects
@@
 			)
 		)
-		(property "Footprint" "Capacitor_SMD:C_0402_1005Metric_Pad0.74x0.62mm_HandSolder"
+		(property "Footprint" "Capacitor_SMD:C_0805_2012Metric_Pad1.18x1.45mm_HandSolder"
 			(at 657.86 276.86 0)
 			(effects
@@
 			)
 		)
-		(property "Value" "470"
+		(property "Value" "820"
 			(at 711.2 386.08 90)
 			(effects
@@
 			)
 		)
-		(property "Value" "1k"
+		(property "Value" "10k"
 			(at 681.99 257.81 90)
 			(effects
@@
 			)
 		)
-		(property "Footprint" "Resistor_SMD:R_0402_1005Metric_Pad0.72x0.64mm_HandSolder"
+		(property "Footprint" "Resistor_SMD:R_0805_2012Metric_Pad1.20x1.40mm_HandSolder"
 			(at 681.99 257.81 0)
 			(effects
@@
 			)
 		)
-		(property "Value" "470"
+		(property "Value" "820"
 			(at 505.46 466.09 90)
 			(effects
@@
 			)
 		)
-		(property "Footprint" "Resistor_SMD:R_0402_1005Metric_Pad0.72x0.64mm_HandSolder"
+		(property "Footprint" "Resistor_SMD:R_0805_2012Metric_Pad1.20x1.40mm_HandSolder"
 			(at 681.99 243.84 0)
 			(effects
@@
 			)
 		)
-		(property "Value" "470"
+		(property "Value" "820"
 			(at 709.93 436.88 90)
 			(effects
@@
 			)
 		)
-		(property "Value" "330"
+		(property "Value" "620"
 			(at 716.28 347.98 90)
 			(effects
@@
 			)
 		)
-		(property "Value" "470"
+		(property "Value" "820"
 			(at 709.93 431.8 90)
 			(effects
@@
 			)
 		)
-		(property "Value" "680"
+		(property "Value" "470"
 			(at 477.52 379.73 90)
 			(effects
@@
 			)
 		)
-		(property "Value" "680"
+		(property "Value" "470"
 			(at 509.27 430.53 90)
 			(effects
@@
 			)
 		)
-		(property "Value" "330"
+		(property "Value" "620"
 			(at 505.46 342.9 90)
 			(effects
@@
 			)
 		)
-		(property "Value" "330"
+		(property "Value" "620"
 			(at 715.01 375.92 90)
 			(effects
@@
 			)
 		)
-		(property "Value" "470"
+		(property "Value" "820"
 			(at 715.01 439.42 90)
 			(effects
@@
 			)
 		)
-		(property "Value" "680"
+		(property "Value" "470"
 			(at 505.46 422.91 90)
 			(effects
@@
 			)
 		)
-		(property "Value" "330"
+		(property "Value" "620"
 			(at 711.2 340.36 90)
 			(effects
@@
 			)
 		)
-		(property "Value" "330"
+		(property "Value" "620"
 			(at 716.28 332.74 90)
 			(effects
@@
 			)
 		)
-		(property "Value" "470"
+		(property "Value" "820"
 			(at 709.93 426.72 90)
 			(effects
@@
 			)
 		)
-		(property "Value" "680"
+		(property "Value" "470"
 			(at 505.46 427.99 90)
 			(effects
@@
 			)
 		)
-		(property "Value" "680"
+		(property "Value" "470"
 			(at 509.27 387.35 90)
 			(effects
@@
 			)
 		)
-		(property "Value" "470"
+		(property "Value" "820"
 			(at 715.01 480.06 90)
 			(effects
@@
 			)
 		)
-		(property "Value" "470"
+		(property "Value" "820"
 			(at 709.93 467.36 90)
 			(effects
@@
 			)
 		)
-		(property "Value" "680"
+		(property "Value" "470"
 			(at 505.46 384.81 90)
 			(effects

Commit message: Updated 25-02-26
Parts:
- C1, C2, C3, C4, C5, C6, C7, C73, C8: footprint Capacitor_SMD:C_0402_1005Metric_Pad0.74x0.62mm_HandSolder -> Capacitor_SMD:C_0603_1608Metric_Pad1.08x0.95mm_HandSolder
- D1, D2, D3, D4, D5, D53, D54, D55, D56, D57, D58, D59, D60, D61, D62, D63: footprint LED_SMD:LED_0402_1005Metric_Pad0.77x0.64mm_HandSolder -> LED_SMD:LED_0603_1608Metric_Pad1.05x0.95mm_HandSolder
- D10, D11, D12, D13, D15, D17, D18, D19, D20, D21, D22, D23, D24, D25, D26, D27, D28, D6, D7, D8, D9: value BLUE -> RED; footprint LED_SMD:LED_0402_1005Metric_Pad0.77x0.64mm_HandSolder -> LED_SMD:LED_0603_1608Metric_Pad1.05x0.95mm_HandSolder
- D14, D49: value WHITE -> RED; footprint LED_SMD:LED_0402_1005Metric_Pad0.77x0.64mm_HandSolder -> LED_SMD:LED_0603_1608Metric_Pad1.05x0.95mm_HandSolder
- D29, D30, D31, D32, D33, D34, D35, D36, D37, D38, D39, D40, D41, D42, D43, D44, D45, D46, D47, D48, D50, D51, D52: value GREEN -> RED; footprint LED_SMD:LED_0402_1005Metric_Pad0.77x0.64mm_HandSolder -> LED_SMD:LED_0603_1608Metric_Pad1.05x0.95mm_HandSolder
- R1, R2, R3, R4, R5, R53, R54, R55, R56, R57, R58, R59, R60, R61, R62, R63: value 620 -> 470; footprint Resistor_SMD:R_0402_1005Metric_Pad0.72x0.64mm_HandSolder -> Resistor_SMD:R_0603_1608Metric_Pad0.98x0.95mm_HandSolder
- R10, R11, R12, R13, R14, R15, R17, R18, R19, R20, R21, R22, R23, R24, R25, R26, R27, R28, R49, R6, R7, R8, R9: footprint Resistor_SMD:R_0402_1005Metric_Pad0.72x0.64mm_HandSolder -> Resistor_SMD:R_0603_1608Metric_Pad0.98x0.95mm_HandSolder
- R29, R30, R31, R32, R33, R34, R35, R36, R37, R38, R39, R40, R41, R42, R43, R44, R45, R46, R47, R48, R50, R51, R52: value 820 -> 470; footprint Resistor_SMD:R_0402_1005Metric_Pad0.72x0.64mm_HandSolder -> Resistor_SMD:R_0603_1608Metric_Pad0.98x0.95mm_HandSolder

Commit message: Minor corrections
Parts:
- C1, C2, C3, C4, C5, C6, C7, C73, C8: LCSC C141382 -> C14663
- C71: LCSC C1953183 -> C7174
- D1, D2, D3, D4, D5, D53, D54, D55, D56, D57, D58, D59, D60, D61, D62, D63: LCSC C71911 -> C2286
- D10, D11, D12, D13, D15, D17, D18, D19, D20, D21, D22, D23, D24, D25, D26, D27, D28, D6, D7, D8, D9: LCSC C131223 -> C2286
- D14, D49: LCSC C74340 -> C2286
- D29, D30, D31, D32, D33, D34, D35, D36, D37, D38, D39, D40, D41, D42, D43, D44, D45, D46, D47, D48, D50, D51, D52: LCSC C74338 -> C2286
- R1, R2, R3, R4, R5, R53, R54, R55, R56, R57, R58, R59, R60, R61, R62, R63: LCSC C25104 -> C23179
- R10, R11, R12, R13, R14, R15, R17, R18, R19, R20, R21, R22, R23, R24, R25, R26, R27, R49, R6, R7, R8, R9: LCSC C25130 -> C23179
- R28, R29, R30, R31, R32, R33, R34, R35, R36, R37, R38, R39, R40, R41, R42, R43, R44, R45, R46, R47, R48, R50, R51, R52: LCSC C25117 -> C23179
- R71: value 10k -> 1k; LCSC C11702 -> C17513
- R72: value 47k -> 15k; LCSC C25762 -> C17475
Connections:
- net at R13.2: now also D13.2 (A); no longer D13.1 (K)
- net at R6.2: now also D6.2 (A); no longer D6.1 (K)
- net at R60.2: now also D60.1 (K); no longer D60.2 (A)
- net at D51.1 (K): now also R51.2; no longer U7.14 (Q5)
- net at D51.2 (A): now also U7.14 (Q5); no longer R51.2
- net at D26.1 (K): now also R26.2; no longer U4.13 (Q6)
- net at D26.2 (A): now also U4.13 (Q6); no longer R26.2
- net at D8.1 (K): now also U1.19 (Q0); no longer R8.2
- net at D8.2 (A): now also R8.2; no longer U1.19 (Q0)
- net at R5.2: now also D5.1 (K); no longer D5.2 (A)
- net at R7.2: now also D7.2 (A); no longer D7.1 (K)
- net at D20.1 (K): now also R20.2; no longer U3.15 (Q4)
- net at D20.2 (A): now also U3.15 (Q4); no longer R20.2
- net at R1.2: now also D1.1 (K); no longer D1.2 (A)
- net at R50.2: now also D50.1 (K); no longer D50.2 (A)
- net at D24.1 (K): now also U3.19 (Q0); no longer R24.2
- net at D24.2 (A): now also R24.2; no longer U3.19 (Q0)
- net at R45.2: now also D45.1 (K); no longer D45.2 (A)
- net at R10.2: now also D10.2 (A); no longer D10.1 (K)
- net at D17.1 (K): now also U3.12 (Q7); no longer R17.2
- net at D17.2 (A): now also R17.2; no longer U3.12 (Q7)
- net at D44.1 (K): now also R44.2; no longer U6.15 (Q4)
- net at D44.2 (A): now also U6.15 (Q4); no longer R44.2
- net at R61.2: now also D61.1 (K); no longer D61.2 (A)
- net at R47.2: now also D47.1 (K); no longer D47.2 (A)
- net at D37.1 (K): now also R37.2; no longer U5.16 (Q3)
- net at D37.2 (A): now also U5.16 (Q3); no longer R37.2
- net at D52.1 (K): now also R52.2; no longer U7.15 (Q4)
- net at D52.2 (A): now also U7.15 (Q4); no longer R52.2
- net at R43.2: now also D43.1 (K); no longer D43.2 (A)
- net at D36.1 (K): now also R36.2; no longer U5.15 (Q4)
- net at D36.2 (A): now also U5.15 (Q4); no longer R36.2
- net at R30.2: now also D30.1 (K); no longer D30.2 (A)
- net at D25.1 (K): now also U4.12 (Q7); no longer R25.2
- net at D25.2 (A): now also R25.2; no longer U4.12 (Q7)
- net at D28.1 (K): now also R28.2; no longer U4.15 (Q4)
- net at D28.2 (A): now also U4.15 (Q4); no longer R28.2
- net at R29.2: now also D29.1 (K); no longer D29.2 (A)
- net at D31.1 (K): now also R31.2; no longer U4.18 (Q1)
- net at D31.2 (A): now also U4.18 (Q1); no longer R31.2
- net at U8.17 (Q2): now also D61.2 (A); no longer D61.1 (K)
- net at U3.13 (Q6): now also D18.1 (K); no longer D18.2 (A)
- net at U3.14 (Q5): now also D19.1 (K); no longer D19.2 (A)
- net at U3.16 (Q3): now also D21.1 (K); no longer D21.2 (A)
- net at U3.17 (Q2): now also D22.1 (K); no longer D22.2 (A)
- net at U3.18 (Q1): now also D23.1 (K); no longer D23.2 (A)
- net at U7.13 (Q6): now also D50.2 (A); no longer D50.1 (K)
- net at D32.1 (K): now also R32.2; no longer U4.19 (Q0)
- net at D32.2 (A): now also U4.19 (Q0); no longer R32.2
- net at D15.1 (K): now also R15.2; no longer U2.18 (Q1)
- net at D15.2 (A): now also U2.18 (Q1); no longer R15.2
- net at U4.14 (Q5): now also D27.2 (A); no longer D27.1 (K)
- net at U4.16 (Q3): now also D29.2 (A); no longer D29.1 (K)
- net at U4.17 (Q2): now also D30.2 (A); no longer D30.1 (K)
- net at R53.2: now also D53.1 (K); no longer D53.2 (A)
- net at R18.2: now also D18.2 (A); no longer D18.1 (K)
- net at D59.1 (K): now also R59.2; no longer U8.15 (Q4)
- net at D59.2 (A): now also U8.15 (Q4); no longer R59.2
- net at D33.1 (K): now also R33.2; no longer U5.12 (Q7)
- net at D33.2 (A): now also U5.12 (Q7); no longer R33.2
- net at D58.1 (K): now also R58.2; no longer U8.14 (Q5)
- net at D58.2 (A): now also U8.14 (Q5); no longer R58.2
- net at R19.2: now also D19.2 (A); no longer D19.1 (K)
- net at R48.2: now also D48.1 (K); no longer D48.2 (A)
- net at D9.1 (K): now also U2.12 (Q7); no longer R9.2
- net at D9.2 (A): now also R9.2; no longer U2.12 (Q7)
- net at U8.12 (Q7): now also D56.2 (A); no longer D56.1 (K)
- net at U8.13 (Q6): now also D57.2 (A); no longer D57.1 (K)
- net at U8.16 (Q3): now also D60.2 (A); no longer D60.1 (K)
- net at U8.18 (Q1): now also D62.2 (A); no longer D62.1 (K)
- net at U8.19 (Q0): now also D63.2 (A); no longer D63.1 (K)
- net at R63.2: now also D63.1 (K); no longer D63.2 (A)
- net at R22.2: now also D22.2 (A); no longer D22.1 (K)
- net at R21.2: now also D21.2 (A); no longer D21.1 (K)
- net at R56.2: now also D56.1 (K); no longer D56.2 (A)
- net at D54.1 (K): now also R54.2; no longer U7.18 (Q1)
- net at D54.2 (A): now also U7.18 (Q1); no longer R54.2
- net at R2.2: now also D2.1 (K); no longer D2.2 (A)
- net at U2.13 (Q6): now also D10.1 (K); no longer D10.2 (A)
- net at U2.14 (Q5): now also D11.1 (K); no longer D11.2 (A)
- net at U2.15 (Q4): now also D12.1 (K); no longer D12.2 (A)
- net at U2.16 (Q3): now also D13.1 (K); no longer D13.2 (A)
- net at U6.14 (Q5): now also D43.2 (A); no longer D43.1 (K)
- net at U1.13 (Q6): now also D2.2 (A); no longer D2.1 (K)
- net at D55.1 (K): now also R55.2; no longer U7.19 (Q0)
- net at D55.2 (A): now also U7.19 (Q0); no longer R55.2
- net at D38.1 (K): now also R38.2; no longer U5.17 (Q2)
- net at D38.2 (A): now also U5.17 (Q2); no longer R38.2
- net at R4.2: now also D4.1 (K); no longer D4.2 (A)
- net at R57.2: now also D57.1 (K); no longer D57.2 (A)
- net at U5.13 (Q6): now also D34.2 (A); no longer D34.1 (K)
- net at U5.14 (Q5): now also D35.2 (A); no longer D35.1 (K)
- net at U5.18 (Q1): now also D39.2 (A); no longer D39.1 (K)
- net at U5.19 (Q0): now also D40.2 (A); no longer D40.1 (K)
- net at U6.12 (Q7): now also D41.2 (A); no longer D41.1 (K)
- net at U6.13 (Q6): now also D42.2 (A); no longer D42.1 (K)
- net at U6.16 (Q3): now also D45.2 (A); no longer D45.1 (K)
- net at U6.17 (Q2): now also D46.2 (A); no longer D46.1 (K)
- net at U6.18 (Q1): now also D47.2 (A); no longer D47.1 (K)
- net at U6.19 (Q0): now also D48.2 (A); no longer D48.1 (K)
- net at R27.2: now also D27.1 (K); no longer D27.2 (A)
- net at R39.2: now also D39.1 (K); no longer D39.2 (A)
- net at R34.2: now also D34.1 (K); no longer D34.2 (A)
- net at R62.2: now also D62.1 (K); no longer D62.2 (A)
- net at U1.16 (Q3): now also D5.2 (A); no longer D5.1 (K)
- net at R23.2: now also D23.2 (A); no longer D23.1 (K)
- net at U7.17 (Q2): now also D53.2 (A); no longer D53.1 (K)
- net at R42.2: now also D42.1 (K); no longer D42.2 (A)
- net at R46.2: now also D46.1 (K); no longer D46.2 (A)
- net at R12.2: now also D12.2 (A); no longer D12.1 (K)
- net at R35.2: now also D35.1 (K); no longer D35.2 (A)
- net at U1.12 (Q7): now also D1.2 (A); no longer D1.1 (K)
- net at U1.15 (Q4): now also D4.2 (A); no longer D4.1 (K)
- net at D3.1 (K): now also R3.2; no longer U1.14 (Q5)
- net at D3.2 (A): now also U1.14 (Q5); no longer R3.2
- net at R41.2: now also D41.1 (K); no longer D41.2 (A)
- net at U1.17 (Q2): now also D6.1 (K); no longer D6.2 (A)
- net at U1.18 (Q1): now also D7.1 (K); no longer D7.2 (A)
- net at R40.2: now also D40.1 (K); no longer D40.2 (A)
- net at R11.2: now also D11.2 (A); no longer D11.1 (K)
Other:
- moved on the sheet: D1, D10, D11, D12, D13, D15, D17, D18, D19, D2, D20, D21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
